Commit message: pumpkin model correct forearm

File: pumpkin_description/robots/pumpkin_description.URDF (robot description, URDF)
Before this commit: robot pumpkin_description, 18 links, 17 joints
Links:
- link base_link: mass 13.9816322818673 -> 13.982
- link chest_link: mass 10.0220880744242 -> 10.022
- link head_link: mass 2.45570096722737 -> 2.4557
- link l_forearm_link: mass 0.460253382032638 -> 0.365895324563534
- link l_wrist0_link: mass 0.0415918723991329 -> 0.0415918723991328
- link l_wrist1_link: mass 0.0490431894031785 -> 0.0490431894031825
- link neck1_link: mass 0.0415918723991327 -> 0.041592
- link neck2_Link: mass 0.0490431894031824 -> 0.049043
- link r_forerarm_link: mass 0.460253382032486 -> 0.365895324563383
- link r_shoulder1_link: mass 0.997303293307219 -> 0.9973
- link r_wrist1_link: mass 0.0490431894031785 -> 0.0490431894031824
Joints:
- joint base_chest: origin xyz=-0.225 -0.0975 1.061 rpy=0 0 3.14159265358979 -> xyz=-0.225 -0.0975 1.061 rpy=0 0 3.1416
- joint l_elbow: limit (none) -> lower=-2 upper=2 effort=0 velocity=0; origin xyz=-0.03268503172314 0 0.14623 rpy=0 1.5707963267949 0 -> xyz=-0.032685 0 0.14623 rpy=0 1.5708 0
- joint l_shoulder_0: limit (none) -> lower=-2 upper=2 effort=0 velocity=0; origin xyz=0.173 0.085 0.224320081404336 rpy=1.5707963267949 0 1.5707963267949 -> xyz=0.173 0.085 0.22432 rpy=1.5708 0 1.5708
- joint l_shoulder_1: limit (none) -> lower=-2 upper=2 effort=0 velocity=0; origin xyz=-0.00189312225294776 0.0485600000000002 0.03917 rpy=1.5707963267949 1.5707963267949 0 -> xyz=-0.0018931 0.04856 0.03917 rpy=1.5708 1.5708 0
- joint l_shoulder_2: limit (none) -> lower=-2 upper=2 effort=0 velocity=0; origin xyz=-0.0932771230454184 -0.0886126007953723 0.0575000000000001 rpy=-1.5707963267949 -1.9127232359829E-16 2.33055532814212 -> xyz=-0.093277 -0.088613 0.0575 rpy=-1.5708 -1.9127E-16 2.3306
- joint l_wrist_0: limit (none) -> lower=-2 upper=2 effort=0 velocity=0; origin xyz=-0.174360874635291 0.00159535499161623 0.0415400000000001 rpy=3.14159265358979 1.5707963267949 0 -> xyz=-0.17436 0.0015954 0.04154 rpy=3.1416 1.5708 0
- joint l_wrist_1: limit (none) -> lower=-2 upper=2 effort=0 velocity=0; origin xyz=-0.0186350000000002 -0.00278669492233996 0.0327000000000002 rpy=1.5707963267949 -2.60208521396521E-16 -1.5707963267949 -> xyz=0.0027867 -0.018635 0.0327 rpy=1.5708 -6.6613E-16 -5.1638E-17
- joint neck2_head: origin xyz=-0.0282400000000006 0 0.0178399999999754 rpy=3.14159265358979 2.6791096154082E-16 -1.5707963267949 -> xyz=-0.02824 0 0.01784 rpy=3.1416 2.6791E-16 -1.5708
- joint neck_0: limit (none) -> lower=-2 upper=2 effort=0 velocity=0; origin xyz=0.0692677669529664 0.042992862378663 0.381070081404336 rpy=1.85037170770859E-15 0 0 -> xyz=0.069268 0.042993 0.38107 rpy=1.8504E-15 0 0
- joint neck_1: limit (none) -> lower=-2 upper=2 effort=0 velocity=0; origin xyz=-0.018635 -0.00278669492233989 0.0327000000000001 rpy=0 1.5707963267949 0 -> xyz=-0.018635 -0.0027867 0.0327 rpy=0 1.5708 0
- joint r_elbow: axis 0 0 -1 -> 0 0 1; limit (none) -> lower=-1.53 upper=2.54 effort=0 velocity=0; origin xyz=0.0326850317231399 0 0.14623 rpy=-1.5707963267949 2.34534436753233E-16 1.5707963267949 -> xyz=0.032685 0 0.14623 rpy=-1.5708 2.3453E-16 1.5708
- joint r_shoulder_0: limit (none) -> lower=-1.94 upper=1.94 effort=0 velocity=0; origin xyz=-0.033 0.085 0.224320081404336 rpy=1.5707963267949 0 -1.5707963267949 -> xyz=-0.033 0.085 0.22432 rpy=1.5708 0 -1.5708
- joint r_shoulder_1: axis 0 0 1 -> 0 0 -1; limit (none) -> lower=-0.7 upper=0.7 effort=0 velocity=0; origin xyz=0.00189312225294823 0.04856 0.03917 rpy=1.5707963267949 -0.809952695179625 1.83845377778929E-15 -> xyz=0.0018931 0.04856 0.03917 rpy=1.5708 -0.80995 1.8385E-15
- joint r_shoulder_2: limit (none) -> lower=-1.94 upper=1.94 effort=0 velocity=0; origin xyz=0.128657742492825 0 0.0575 rpy=-1.5707963267949 6.96956074407882E-18 -1.5707963267949 -> xyz=0.12866 0 0.0575 rpy=-1.5708 6.9696E-18 -1.5708
- joint r_wrist_0: limit (none) -> lower=-1.54 upper=1.54 effort=0 velocity=0; origin xyz=0.00159535499161634 -0.174360874635292 0.0415800000000001 rpy=1.5707963267949 -1.28225840869416E-16 2.70187914736707E-17 -> xyz=0.0015954 -0.17436 0.04158 rpy=1.5708 -1.2823E-16 2.7019E-17
- joint r_wrist_1: limit (none) -> lower=-1.75 upper=1 effort=0 velocity=0; origin xyz=0.00278669492233996 0.0186349999999999 0.0327 rpy=1.5707963267949 -5.41724245269373E-16 1.4587432664842E-16 -> xyz=0.018635 -0.0027867 0.0327 rpy=1.5708 -6.6613E-16 -1.5708
